File: 9axis-sensor/main.sch (EAGLE design)
At the start: 9 parts, among them IC1 LPC1114FDH28, IC2 MPU-9250

Commit message: 基板1版できた。
Parts:
- added C2, C3, C4, C5, C6: 1u, rcl:C-EUC0402
- added IC3: RN-42, SparkFun-RF:BLUETOOTH-RN41"
- added IC4: MAX1555, maxim:MAX1555
- added IC5: NJM2866F33, Library:NJM2866F33
- added J1: ZX62R-B-5P, Library:ZX62R-B-5P
- added J2: 53261-02, con-molex:53261-02
- added LED1, LED3: Status LED, led:LEDCHIP-LED0603
- added LED2: Activity LED, led:LEDCHIP-LED0603
- added R2, R3, R4: 1k, rcl:R-US_R0402
- added SW1: SK-12D01-VG4, Library:SK-12D01-VG4
- C1: MF (none) -> Murata; MPN (none) -> GRM155R61E105KA12D; OC (none) -> 846-7287; SITE (none) -> RS Components
- IC2: device ic-package:DIL10 -> Library:MPU-9250; MF InvenSense -> (none); MPN MPU-9250 -> (none); OC 12250 -> (none); SITE StrawberryLinux -> (none)
- TP1: value PTR1B1,27 -> 3V3
- TP2: value PTR1B1,27 -> SWDIO
- TP3: value PTR1B1,27 -> SWCLK
- TP4: value PTR1B1,27 -> RESET
- TP5: value PTR1B1,27 -> GND
Connections:
- new net ACTIVITY: IC3.PIO8, R3.1
- new net BATT: C4.1, IC4.BAT, J2-1.S, R4.2, SW1.P$1
- new net N$1: IC3.UARTCTS, IC3.UARTRTS
- new net N$2: C3.1, IC4.USB, J1.VBUS
- new net N$3: LED1.C, R2.2
- new net N$4: LED2.C, R3.2
- new net N$5: IC4.!CHG, LED3.C
- new net N$6: LED3.A, R4.1
- new net N$7: C5.1, IC5.CONTROL, IC5.VIN, SW1.P$3
- new net STATUS: IC3.PIO5, R2.1
- net +3V3: now also C2.1, C6.1, IC2.VDD, IC2.VDDIO, IC3.VDD, IC5.VOUT, LED1.A, LED2.A; no longer IC2.1, IC2.2
- net CS: now also IC2./CS; no longer IC2.6
- net GND: now also C2.2, C3.2, C4.2, C5.2, C6.2, IC2.GND, IC3.GND, IC3.GND1, IC3.GND2, IC3.GND3, IC4.GND, IC5.GND, J1.GND, J1.SHEILDS, J2-2.S; no longer IC2.10
- net MISO: now also IC2.AD0/SDO; no longer IC2.5
- net MOSI: now also IC2.SDA/SDI; no longer IC2.4
- net RX: now also IC3.UARTTX
- net SCK: now also IC2.SCL/SCLK; no longer IC2.3
- net TX: now also IC3.UARTRX

Commit message: バッテリ電圧測定回路を追加。基板更新。
Parts:
- added R5, R6: 10k, rcl:R-US_R0402
Connections:
- new net N$8: IC1.TMS/PIO1_0/AD1/CT32B1_CAP0, R5.1, R6.2
- net +3V3: now also R5.2
- net GND: now also R6.1
Changed lines of the file:
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@@
 </variantdefs>
 <classes>
-<class number="0" name="default" width="0" drill="0">
+<class number="0" name="default" width="0.254" drill="0">
 </class>
 </classes>
@@
 <part name="GND14" library="supply1" deviceset="GND" device=""/>
 <part name="IC2" library="Library" deviceset="MPU-9250" device=""/>
+<part name="R5" library="rcl" deviceset="R-US_" device="R0402" value="10k"/>
+<part name="R6" library="rcl" deviceset="R-US_" device="R0402" value="10k"/>
+<part name="GND15" library="supply1" deviceset="GND" device=""/>
+<part name="+3V9" library="supply1" deviceset="+3V3" device=""/>
 </parts>
 <sheets>
@@
 </instance>
 <instance part="IC2" gate="G$1" x="55.88" y="81.28"/>
+<instance part="R5" gate="G$1" x="172.72" y="160.02"/>
+<instance part="R6" gate="G$1" x="165.1" y="152.4" rot="R90"/>
+<instance part="GND15" gate="1" x="165.1" y="142.24"/>
+<instance part="+3V9" gate="G$1" x="182.88" y="167.64"/>
 </instances>
 <busses>
@@
 <wire x1="119.38" y1="66.04" x2="132.08" y2="66.04" width="0.1524" layer="91"/>
 <junction x="132.08" y="66.04"/>
+</segment>
+<segment>
+<pinref part="R5" gate="G$1" pin="2"/>
+<pinref part="+3V9" gate="G$1" pin="+3V3"/>
+<wire x1="177.8" y1="160.02" x2="182.88" y2="160.02" width="0.1524" layer="91"/>
+<wire x1="182.88" y1="160.02" x2="182.88" y2="165.1" width="0.1524" layer="91"/>
 </segment>
 </net>
@@
 <junction x="213.36" y="38.1"/>
 </segment>
+<segment>
+<pinref part="GND15" gate="1" pin="GND"/>
+<pinref part="R6" gate="G$1" pin="1"/>
+<wire x1="165.1" y1="144.78" x2="165.1" y2="147.32" width="0.1524" layer="91"/>
+</segment>
 </net>
 <net name="SWDIO" class="0">
@@
 </segment>
 </net>
+<net name="N$8" class="0">
+<segment>
+<pinref part="IC1" gate="G$1" pin="TMS/PIO1_0/AD1/CT32B1_CAP0"/>
+<wire x1="134.62" y1="160.02" x2="165.1" y2="160.02" width="0.1524" layer="91"/>
+<pinref part="R5" gate="G$1" pin="1"/>
+<pinref part="R6" gate="G$1" pin="2"/>
+<wire x1="165.1" y1="160.02" x2="167.64" y2="160.02" width="0.1524" layer="91"/>
+<wire x1="165.1" y1="160.02" x2="165.1" y2="157.48" width="0.1524" layer="91"/>
+<junction x="165.1" y="160.02"/>
+</segment>
+</net>

Commit message: 部品番号を記載
Parts:
- J2: MF (none) -> Molex; MPN (none) -> 53261-0271; OC (none) -> 542-7090; SITE (none) -> RS Components
- LED1: MF (none) -> OptoSupply; MPN (none) -> OSYG1608C1A; OC (none) -> I-03980; SITE (none) -> Akizukidenshi
- LED2: MF (none) -> OptoSupply; MPN (none) -> OSBL1608C1A; OC (none) -> I-03982; SITE (none) -> Akizukidenshi
- LED3: MF (none) -> OptoSupply; MPN (none) -> OSHR1608C1A; OC (none) -> I-03978; SITE (none) -> Akizukidenshi
Changed lines of the file:
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@@
 <part name="LED1" library="led" deviceset="LED" device="CHIP-LED0603" value="Status LED">
 <attribute name="COLOR" value="Green"/>
+<attribute name="MF" value="OptoSupply"/>
+<attribute name="MPN" value="OSYG1608C1A"/>
+<attribute name="OC" value="I-03980"/>
+<attribute name="SITE" value="Akizukidenshi"/>
 </part>
 <part name="LED2" library="led" deviceset="LED" device="CHIP-LED0603" value="Activity LED">
 <attribute name="COLOR" value="Blue"/>
+<attribute name="MF" value="OptoSupply"/>
+<attribute name="MPN" value="OSBL1608C1A"/>
+<attribute name="OC" value="I-03982"/>
+<attribute name="SITE" value="Akizukidenshi"/>
 </part>
 <part name="R2" library="rcl" deviceset="R-US_" device="R0402" value="1k"/>
@@
 <part name="LED3" library="led" deviceset="LED" device="CHIP-LED0603" value="Status LED">
 <attribute name="COLOR" value="Red"/>
+<attribute name="MF" value="OptoSupply"/>
+<attribute name="MPN" value="OSHR1608C1A"/>
+<attribute name="OC" value="I-03978"/>
+<attribute name="SITE" value="Akizukidenshi"/>
 </part>
 <part name="R4" library="rcl" deviceset="R-US_" device="R0402" value="1k"/>
@@
 <part name="GND12" library="supply1" deviceset="GND" device=""/>
 <part name="GND13" library="supply1" deviceset="GND" device=""/>
-<part name="J2" library="con-molex" deviceset="53?-02" device="261"/>
+<part name="J2" library="con-molex" deviceset="53?-02" device="261">
+<attribute name="MF" value="Molex"/>
+<attribute name="MPN" value="53261-0271"/>
+<attribute name="OC" value="542-7090"/>
+<attribute name="SITE" value="RS Components"/>
+</part>
 <part name="GND14" library="supply1" deviceset="GND" device=""/>
 <part name="IC2" library="Library" deviceset="MPU-9250" device=""/>
@@
 <instance part="LED1" gate="G$1" x="116.84" y="66.04" rot="R270">
 <attribute name="COLOR" x="112.268" y="58.166" size="1.778" layer="96" display="both"/>
+<attribute name="MF" x="116.84" y="66.04" size="1.778" layer="96" rot="R270" display="off"/>
+<attribute name="MPN" x="116.84" y="66.04" size="1.778" layer="96" rot="R270" display="off"/>
+<attribute name="OC" x="116.84" y="66.04" size="1.778" layer="96" rot="R270" display="off"/>
+<attribute name="SITE" x="116.84" y="66.04" size="1.778" layer="96" rot="R270" display="off"/>
 </instance>
 <instance part="LED2" gate="G$1" x="116.84" y="53.34" rot="R270">
 <attribute name="COLOR" x="112.014" y="45.466" size="1.778" layer="96" display="both"/>
+<attribute name="MF" x="116.84" y="53.34" size="1.778" layer="96" rot="R270" display="off"/>
+<attribute name="MPN" x="116.84" y="53.34" size="1.778" layer="96" rot="R270" display="off"/>
+<attribute name="OC" x="116.84" y="53.34" size="1.778" layer="96" rot="R270" display="off"/>
+<attribute name="SITE" x="116.84" y="53.34" size="1.778" layer="96" rot="R270" display="off"/>
 </instance>
 <instance part="R2" gate="G$1" x="101.6" y="66.04"/>
@@
 <instance part="LED3" gate="G$1" x="124.46" y="139.7" rot="R270">
 <attribute name="COLOR" x="119.888" y="131.826" size="1.778" layer="96" display="both"/>
+<attribute name="MF" x="124.46" y="139.7" size="1.778" layer="96" rot="R270" display="off"/>
+<attribute name="MPN" x="124.46" y="139.7" size="1.778" layer="96" rot="R270" display="off"/>
+<attribute name="OC" x="124.46" y="139.7" size="1.778" layer="96" rot="R270" display="off"/>
+<attribute name="SITE" x="124.46" y="139.7" size="1.778" layer="96" rot="R270" display="off"/>
 </instance>
 <instance part="R4" gate="G$1" x="137.16" y="139.7"/>
@@
 <instance part="GND12" gate="1" x="91.44" y="43.18"/>
 <instance part="GND13" gate="1" x="152.4" y="43.18"/>
-<instance part="J2" gate="-1" x="210.82" y="111.76"/>
+<instance part="J2" gate="-1" x="210.82" y="111.76">
+<attribute name="OC" x="210.82" y="111.76" size="1.778" layer="96" display="off"/>
+<attribute name="SITE" x="210.82" y="111.76" size="1.778" layer="96" display="off"/>
+</instance>
 <instance part="J2" gate="-2" x="210.82" y="109.22"/>
 <instance part="GND14" gate="1" x="205.74" y="99.06"/>

Commit message: ADCの配線ミスを修正
Connections:
- net +3V3: no longer R5.2
- net BATT: now also R5.2
Changed lines of the file:
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@@
 <part name="R6" library="rcl" deviceset="R-US_" device="R0402" value="10k"/>
 <part name="GND15" library="supply1" deviceset="GND" device=""/>
-<part name="+3V9" library="supply1" deviceset="+3V3" device=""/>
 </parts>
 <sheets>
@@
 <instance part="R6" gate="G$1" x="165.1" y="152.4" rot="R90"/>
 <instance part="GND15" gate="1" x="165.1" y="142.24"/>
-<instance part="+3V9" gate="G$1" x="182.88" y="167.64"/>
 </instances>
 <busses>
@@
 <wire x1="119.38" y1="66.04" x2="132.08" y2="66.04" width="0.1524" layer="91"/>
 <junction x="132.08" y="66.04"/>
-</segment>
-<segment>
-<pinref part="R5" gate="G$1" pin="2"/>
-<pinref part="+3V9" gate="G$1" pin="+3V3"/>
-<wire x1="177.8" y1="160.02" x2="182.88" y2="160.02" width="0.1524" layer="91"/>
-<wire x1="182.88" y1="160.02" x2="182.88" y2="165.1" width="0.1524" layer="91"/>
 </segment>
 </net>
@@
 </segment>
 </net>
+<net name="BATT" class="0">
+<segment>
+<pinref part="R5" gate="G$1" pin="2"/>
+<wire x1="177.8" y1="160.02" x2="185.42" y2="160.02" width="0.1524" layer="91"/>
+<label x="185.42" y="160.02" size="1.778" layer="95" xref="yes"/>
+</segment>
+</net>

Commit message: チップ部品サイズを1608に変更
Parts:
- C1, C2, C5: value 1u -> 0.1u; device rcl:C-EUC0402 -> rcl:C-EUC0603; MF Murata -> (none); MPN GRM155R61E105KA12D -> (none); OC 846-7287 -> (none); SITE RS Components -> (none)
- C3, C4, C6: device rcl:C-EUC0402 -> rcl:C-EUC0603; MF Murata -> (none); MPN GRM155R61E105KA12D -> (none); OC 846-7287 -> (none); SITE RS Components -> (none)
- LED3: value Status LED -> Charge LED
- R1, R2, R3, R4, R5, R6: device rcl:R-US_R0402 -> rcl:R-US_R0603
Changed lines of the file:
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@@
 <part name="GND2" library="supply1" deviceset="GND" device=""/>
 <part name="+3V2" library="supply1" deviceset="+3V3" device=""/>
-<part name="R1" library="rcl" deviceset="R-US_" device="R0402" value="10k"/>
+<part name="R1" library="rcl" deviceset="R-US_" device="R0603" value="10k"/>
 <part name="+3V3" library="supply1" deviceset="+3V3" device=""/>
 <part name="+3V4" library="supply1" deviceset="+3V3" device=""/>
@@
 <part name="+3V5" library="supply1" deviceset="+3V3" device=""/>
 <part name="GND4" library="supply1" deviceset="GND" device=""/>
-<part name="C1" library="rcl" deviceset="C-EU" device="C0402" value="1u">
-<attribute name="MF" value="Murata"/>
-<attribute name="MPN" value="GRM155R61E105KA12D"/>
-<attribute name="OC" value="846-7287"/>
-<attribute name="SITE" value="RS Components"/>
-</part>
+<part name="C1" library="rcl" deviceset="C-EU" device="C0603" value="0.1u"/>
 <part name="IC3" library="SparkFun-RF" deviceset="BLUETOOTH-RN41" device="&quot;" value="RN-42">
 <attribute name="MF" value="Microchip"/>
@@
 <attribute name="SITE" value="Akizukidenshi"/>
 </part>
-<part name="R2" library="rcl" deviceset="R-US_" device="R0402" value="1k"/>
-<part name="R3" library="rcl" deviceset="R-US_" device="R0402" value="1k"/>
+<part name="R2" library="rcl" deviceset="R-US_" device="R0603" value="1k"/>
+<part name="R3" library="rcl" deviceset="R-US_" device="R0603" value="1k"/>
 <part name="+3V7" library="supply1" deviceset="+3V3" device=""/>
 <part name="FRAME2" library="frames" deviceset="A4L-LOC" device=""/>
@@
 <part name="GND9" library="supply1" deviceset="GND" device=""/>
 <part name="GND10" library="supply1" deviceset="GND" device=""/>
-<part name="C2" library="rcl" deviceset="C-EU" device="C0402" value="1u">
-<attribute name="MF" value="Murata"/>
-<attribute name="MPN" value="GRM155R61E105KA12D"/>
-<attribute name="OC" value="846-7287"/>
-<attribute name="SITE" value="RS Components"/>
-</part>
-<part name="C3" library="rcl" deviceset="C-EU" device="C0402" value="1u">
-<attribute name="MF" value="Murata"/>
-<attribute name="MPN" value="GRM155R61E105KA12D"/>
-<attribute name="OC" value="846-7287"/>
-<attribute name="SITE" value="RS Components"/>
-</part>
-<part name="C4" library="rcl" deviceset="C-EU" device="C0402" value="1u">
-<attribute name="MF" value="Murata"/>
-<attribute name="MPN" value="GRM155R61E105KA12D"/>
-<attribute name="OC" value="846-7287"/>
-<attribute name="SITE" value="RS Components"/>
-</part>
-<part name="LED3" library="led" deviceset="LED" device="CHIP-LED0603" value="Status LED">
+<part name="C2" library="rcl" deviceset="C-EU" device="C0603" value="0.1u"/>
+<part name="C3" library="rcl" deviceset="C-EU" device="C0603" value="1u"/>
+<part name="C4" library="rcl" deviceset="C-EU" device="C0603" value="1u"/>
+<part name="LED3" library="led" deviceset="LED" device="CHIP-LED0603" value="Charge LED">
 <attribute name="COLOR" value="Red"/>
 <attribute name="MF" value="OptoSupply"/>
@@
 <attribute name="SITE" value="Akizukidenshi"/>
 </part>
-<part name="R4" library="rcl" deviceset="R-US_" device="R0402" value="1k"/>
+<part name="R4" library="rcl" deviceset="R-US_" device="R0603" value="1k"/>
 <part name="IC5" library="Library" deviceset="NJM2866F33" device=""/>
 <part name="SW1" library="Library" deviceset="SK-12D01-VG4" device=""/>
 <part name="GND11" library="supply1" deviceset="GND" device=""/>
 <part name="+3V8" library="supply1" deviceset="+3V3" device=""/>
-<part name="C5" library="rcl" deviceset="C-EU" device="C0402" value="1u">
-<attribute name="MF" value="Murata"/>
-<attribute name="MPN" value="GRM155R61E105KA12D"/>
-<attribute name="OC" value="846-7287"/>
-<attribute name="SITE" value="RS Components"/>
-</part>
-<part name="C6" library="rcl" deviceset="C-EU" device="C0402" value="1u">
-<attribute name="MF" value="Murata"/>
-<attribute name="MPN" value="GRM155R61E105KA12D"/>
-<attribute name="OC" value="846-7287"/>
-<attribute name="SITE" value="RS Components"/>
-</part>
+<part name="C5" library="rcl" deviceset="C-EU" device="C0603" value="0.1u"/>
+<part name="C6" library="rcl" deviceset="C-EU" device="C0603" value="1u"/>
 <part name="GND12" library="supply1" deviceset="GND" device=""/>
 <part name="GND13" library="supply1" deviceset="GND" device=""/>
@@
 <part name="GND14" library="supply1" deviceset="GND" device=""/>
 <part name="IC2" library="Library" deviceset="MPU-9250" device=""/>
-<part name="R5" library="rcl" deviceset="R-US_" device="R0402" value="10k"/>
-<part name="R6" library="rcl" deviceset="R-US_" device="R0402" value="10k"/>
+<part name="R5" library="rcl" deviceset="R-US_" device="R0603" value="10k"/>
+<part name="R6" library="rcl" deviceset="R-US_" device="R0603" value="10k"/>
 <part name="GND15" library="supply1" deviceset="GND" device=""/>
 </parts>
@@
 <instance part="+3V5" gate="G$1" x="132.08" y="104.14"/>
 <instance part="GND4" gate="1" x="132.08" y="81.28"/>
-<instance part="C1" gate="G$1" x="132.08" y="93.98">
-<attribute name="MF" x="132.08" y="93.98" size="1.778" layer="96" display="off"/>
-<attribute name="MPN" x="132.08" y="93.98" size="1.778" layer="96" display="off"/>
-<attribute name="OC" x="132.08" y="93.98" size="1.778" layer="96" display="off"/>
-<attribute name="SITE" x="132.08" y="93.98" size="1.778" layer="96" display="off"/>
-</instance>
+<instance part="C1" gate="G$1" x="132.08" y="93.98"/>
 <instance part="IC3" gate="G$1" x="187.96" y="66.04">
 <attribute name="MF" x="187.96" y="66.04" size="1.778" layer="96" display="off"/>
@@
 <instance part="R3" gate="G$1" x="101.6" y="53.34"/>
 <instance part="+3V7" gate="G$1" x="132.08" y="73.66"/>
-<instance part="C2" gate="G$1" x="139.7" y="93.98">
-<attribute name="MF" x="139.7" y="93.98" size="1.778" layer="96" display="off"/>
-<attribute name="MPN" x="139.7" y="93.98" size="1.778" layer="96" display="off"/>
-<attribute name="OC" x="139.7" y="93.98" size="1.778" layer="96" display="off"/>
-<attribute name="SITE" x="139.7" y="93.98" size="1.778" layer="96" display="off"/>
-</instance>
+<instance part="C2" gate="G$1" x="139.7" y="93.98"/>
 <instance part="IC2" gate="G$1" x="55.88" y="81.28"/>
 <instance part="R5" gate="G$1" x="172.72" y="160.02"/>
@@
 <instance part="GND9" gate="1" x="73.66" y="101.6"/>
 <instance part="GND10" gate="1" x="132.08" y="101.6"/>
-<instance part="C3" gate="G$1" x="73.66" y="111.76">
-<attribute name="MF" x="73.66" y="111.76" size="1.778" layer="96" display="off"/>
-<attribute name="MPN" x="73.66" y="111.76" size="1.778" layer="96" display="off"/>
-<attribute name="OC" x="73.66" y="111.76" size="1.778" layer="96" display="off"/>
-<attribute name="SITE" x="73.66" y="111.76" size="1.778" layer="96" display="off"/>
-</instance>
-<instance part="C4" gate="G$1" x="132.08" y="114.3">
-<attribute name="MF" x="132.08" y="114.3" size="1.778" layer="96" display="off"/>
-<attribute name="MPN" x="132.08" y="114.3" size="1.778" layer="96" display="off"/>
-<attribute name="OC" x="132.08" y="114.3" size="1.778" layer="96" display="off"/>
-<attribute name="SITE" x="132.08" y="114.3" size="1.778" layer="96" display="off"/>
-</instance>
+<instance part="C3" gate="G$1" x="73.66" y="111.76"/>
+<instance part="C4" gate="G$1" x="132.08" y="114.3"/>
 <instance part="LED3" gate="G$1" x="124.46" y="139.7" rot="R270">
 <attribute name="COLOR" x="119.888" y="131.826" size="1.778" layer="96" display="both"/>
@@
 <instance part="GND11" gate="1" x="99.06" y="43.18"/>
 <instance part="+3V8" gate="G$1" x="157.48" y="73.66"/>
-<instance part="C5" gate="G$1" x="91.44" y="55.88">
-<attribute name="MF" x="91.44" y="55.88" size="1.778" layer="96" display="off"/>
-<attribute name="MPN" x="91.44" y="55.88" size="1.778" layer="96" display="off"/>
-<attribute name="OC" x="91.44" y="55.88" size="1.778" layer="96" display="off"/>
-<attribute name="SITE" x="91.44" y="55.88" size="1.778" layer="96" display="off"/>
-</instance>
-<instance part="C6" gate="G$1" x="152.4" y="55.88">
-<attribute name="MF" x="152.4" y="55.88" size="1.778" layer="96" display="off"/>
-<attribute name="MPN" x="152.4" y="55.88" size="1.778" layer="96" display="off"/>
-<attribute name="OC" x="152.4" y="55.88" size="1.778" layer="96" display="off"/>
-<attribute name="SITE" x="152.4" y="55.88" size="1.778" layer="96" display="off"/>
-</instance>
+<instance part="C5" gate="G$1" x="91.44" y="55.88"/>
+<instance part="C6" gate="G$1" x="152.4" y="55.88"/>
 <instance part="GND12" gate="1" x="91.44" y="43.18"/>
 <instance part="GND13" gate="1" x="152.4" y="43.18"/>
